Commit message: feat: add throw_in_cup task

File: assets/mjcf/bucket/100454/mobility.urdf (robot description, URDF)
Before this commit: robot partnet_75612c0c1d5730eaf93a86670701266, 2 links, 1 joints
Links:
- link link_1: geometry collision mesh filename=textured_objs/original-1.obj scale=0.13 0.13 0.13; visual mesh filename=textured_objs/original-1.obj scale=0.13 0.13 0.13
